Commit message: modify for mbzirc2020

File: urdf/sample_robot.gazebo.xacro (robot description, xacro)
@@ -2,6 +2,24 @@
 <robot
     xmlns:xacro="http://www.ros.org/wiki/xacro" name="sample_robot" >
+  <xacro:arg name="robot_name" default="hydrus" />
+  <!-- gazebo for Realsense D435 -->
+  <!--  The following values model the aluminum peripherial case for the
+        D435 camera, with the camera joint represented by the actual
+        peripherial camera tripod mount -->
+  <xacro:property name="d435_cam_depth_to_left_ir_offset" value="0.0"/>
+  <xacro:property name="d435_cam_depth_to_right_ir_offset" value="-0.050"/>
+  <xacro:property name="d435_cam_depth_to_color_offset" value="0.015"/>
+  <xacro:property name="d435_cam_width" value="0.090"/>
+  <xacro:property name="d435_cam_height" value="0.025"/>
+  <xacro:property name="d435_cam_depth" value="0.02505"/>
+  <xacro:property name="d435_cam_mount_from_center_offset" value="0.0149"/>
+  <!--  The following offset is relative the the physical D435 camera peripherial
+        camera tripod mount -->
+  <xacro:property name="d435_cam_depth_px" value="${d435_cam_mount_from_center_offset}"/>
+  <xacro:property name="d435_cam_depth_py" value="0.0175"/>
+  <xacro:property name="d435_cam_depth_pz" value="${d435_cam_height/2}"/>
   <link name="base_link">
     <visual>
+      <origin xyz="0 0 0.5" rpy="0 0 0"/>
       <geometry>
         <box size="0.5 0.5 1.0"/>
@@ -9,4 +27,5 @@
     </visual>
     <collision>
+      <origin xyz="0 0 0.5" rpy="0 0 0"/>
       <geometry>
         <box size="0.5 0.5 1.0"/>
@@ -24,7 +43,107 @@
     <origin xyz="-2.0 0.0 1.0" rpy="0.0 1.57 0.0"/>
     <parent link="base_link"/>
-    <child link="camera_link"/>
+    <child link="rs_d435_link"/>
   </joint>
-  <link name="camera_link"/>
+  <link name="rs_d435_link"/>
+    <!-- camera depth joints and links -->
+  <joint name="rs_d435_depth_joint" type="fixed">
+    <origin xyz="0 0 0" rpy="0 0 0"/>
+    <parent link="rs_d435_link"/>
+    <child link="rs_d435_depth_frame" />
+  </joint>
+  <link name="rs_d435_depth_frame"/>
+  <joint name="rs_d435_depth_optical_joint" type="fixed">
+    <origin xyz="0 0 0" rpy="${-pi/2} 0 ${-pi/2}" />
+    <parent link="rs_d435_depth_frame" />
+    <child link="rs_d435_depth_optical_frame" />
+  </joint>
+  <link name="rs_d435_depth_optical_frame"/>
+  <!-- camera left IR joints and links -->
+  <joint name="rs_d435_left_ir_joint" type="fixed">
+    <origin xyz="0 ${d435_cam_depth_to_left_ir_offset} 0" rpy="0 0 0" />
+    <parent link="rs_d435_depth_frame" />
+    <child link="rs_d435_left_ir_frame" />
+  </joint>
+  <link name="rs_d435_left_ir_frame"/>
+  <joint name="rs_d435_left_ir_optical_joint" type="fixed">
+    <origin xyz="0 0 0" rpy="${-pi/2} 0 ${-pi/2}" />
+    <parent link="rs_d435_left_ir_frame" />
+    <child link="rs_d435_left_ir_optical_frame" />
+  </joint>
+  <link name="rs_d435_left_ir_optical_frame"/>
+  <!-- camera right IR joints and links -->
+  <joint name="rs_d435_right_ir_joint" type="fixed">
+    <origin xyz="0 ${d435_cam_depth_to_right_ir_offset} 0" rpy="0 0 0" />
+    <parent link="rs_d435_depth_frame" />
+    <child link="rs_d435_right_ir_frame" />
+  </joint>
+  <link name="rs_d435_right_ir_frame"/>
+  <joint name="rs_d435_right_ir_optical_joint" type="fixed">
+    <origin xyz="0 0 0" rpy="${-pi/2} 0 ${-pi/2}" />
+    <parent link="rs_d435_right_ir_frame" />
+    <child link="rs_d435_right_ir_optical_frame" />
+  </joint>
+  <link name="rs_d435_right_ir_optical_frame"/>
+  <!-- camera color joints and links -->
+  <joint name="rs_d435_color_joint" type="fixed">
+    <origin xyz="0 ${d435_cam_depth_to_color_offset} 0" rpy="0 0 0" />
+    <parent link="rs_d435_depth_frame" />
+    <child link="rs_d435_color_frame" />
+  </joint>
+  <link name="rs_d435_color_frame"/>
+  <joint name="rs_d435_color_optical_joint" type="fixed">
+    <origin xyz="0 0 0" rpy="${-pi/2} 0 ${-pi/2}" />
+    <parent link="rs_d435_color_frame" />
+    <child link="rs_d435_color_optical_frame" />
+  </joint>
+  <link name="rs_d435_color_optical_frame"/>
+  <!-- gazebo plugin -->
+  <gazebo reference="rs_d435_color_frame">
+    <sensor type="depth" name="rs_d435_camera">
+      <update_rate>20.0</update_rate>
+      <camera name="head">
+	<horizontal_fov>0.95725190791890935</horizontal_fov>
+	<!--vertical_fov>0.74223480644853568</vertical_fov-->
+	<image>
+	  <width>640</width>
+	  <height>480</height>
+	  <format>B8G8R8</format>
+	</image>
+	<clip>
+	  <near>0.02</near>
+	  <far>300</far>
+	</clip>
+	<noise>
+	  <type>gaussian</type>
+	  <mean>0.0</mean>
+	  <stddev>0.007</stddev>
+	</noise>
+      </camera>
+      <plugin name="depth_camera" filename="libgazebo_ros_openni_kinect.so">
+        <robotNamespace>$(arg robot_name)</robotNamespace>
+	<baseline>0.06</baseline>
+	<alwaysOn>true</alwaysOn>
+	<updateRate>0.0</updateRate>
+	<cameraName>rs_d435</cameraName>
+	<imageTopicName>color/image_rect_color</imageTopicName>
+	<cameraInfoTopicName>color/camera_info</cameraInfoTopicName>
+	<depthImageCameraInfoTopicName>aligned_depth_to_color/camera_info</depthImageCameraInfoTopicName>
+	<depthImageTopicName>aligned_depth_to_color/image_raw</depthImageTopicName>
+	<pointCloudTopicName>depth_registered/points</pointCloudTopicName>
+	<frameName>rs_d435_color_optical_frame</frameName>
+	<pointCloudCutoff>0.05</pointCloudCutoff>
+	<distortionK1>0</distortionK1>
+	<distortionK2>0</distortionK2>
+	<distortionK3>0</distortionK3>
+	<distortionT1>0</distortionT1>
+	<distortionT2>0</distortionT2>
+	<CxPrime>0</CxPrime>
+	<Cx>0</Cx>
+	<Cy>0</Cy>
+	<focalLength>0</focalLength>
+	<hackBaseline>0</hackBaseline>
+      </plugin>
+    </sensor>
+  </gazebo>
   <gazebo>
     <plugin name="gazebo_ros_control" filename="libgazebo_ros_control.so">
@@ -32,50 +151,3 @@
     </plugin>
   </gazebo>
-  <!-- gazebo plugin -->
-  <gazebo reference="camera_link">
-    <sensor type="depth" name="camera">
-      <update_rate>20.0</update_rate>
-      <camera name="head">
-        <horizontal_fov>1.59174</horizontal_fov>
-        <vertical_fov>1.14319</vertical_fov>
-        <image>
-          <width>1280</width>
-          <height>720</height>
-          <format>R8G8B8</format>
-        </image>
-        <clip>
-          <near>0.02</near>
-          <far>300</far>
-        </clip>
-        <noise>
-          <type>gaussian</type>
-          <mean>0.0</mean>
-          <stddev>0.007</stddev>
-        </noise>
-      </camera>
-      <plugin name="depth_camera" filename="libgazebo_ros_openni_kinect.so">
-        <baseline>0.06</baseline>
-        <alwaysOn>true</alwaysOn>
-        <updateRate>0.0</updateRate>
-        <cameraName>camera</cameraName>
-        <imageTopicName>color/image_rect_color</imageTopicName>
-        <cameraInfoTopicName>color/camera_info</cameraInfoTopicName>
-        <depthImageCameraInfoTopicName>aligned_depth_to_color/camera_info</depthImageCameraInfoTopicName>
-        <depthImageTopicName>aligned_depth_to_color/image_raw</depthImageTopicName>
-        <pointCloudTopicName>depth_registered/points</pointCloudTopicName>
-        <frameName>camera_color_optical_frame</frameName>
-        <pointCloudCutoff>0.05</pointCloudCutoff>
-        <distortionK1>0</distortionK1>
-        <distortionK2>0</distortionK2>
-        <distortionK3>0</distortionK3>
-        <distortionT1>0</distortionT1>
-        <distortionT2>0</distortionT2>
-        <CxPrime>0</CxPrime>
-        <Cx>0</Cx>
-        <Cy>0</Cy>
-        <focalLength>0</focalLength>
-        <hackBaseline>0</hackBaseline>
-      </plugin>
-    </sensor>
-  </gazebo>
 </robot>

Commit message: add pitch joint

File: urdf/sample_robot.gazebo.xacro (robot description, xacro)
@@ -19,4 +19,9 @@
   <xacro:property name="d435_cam_depth_py" value="0.0175"/>
   <xacro:property name="d435_cam_depth_pz" value="${d435_cam_height/2}"/>
+  <link name="world"/>
+  <joint name="fixed" type="fixed">
+    <parent link="world"/>
+    <child link="base_link"/>
+  </joint>
   <link name="base_link">
     <visual>
@@ -40,10 +45,29 @@
     </inertial>
   </link>
-  <joint name="joint1" type="fixed">
+  <joint name="joint1" type="continuous">
     <origin xyz="-2.0 0.0 1.0" rpy="0.0 1.57 0.0"/>
+    <axis xyz="0 1 0"/>
     <parent link="base_link"/>
     <child link="rs_d435_link"/>
   </joint>
-  <link name="rs_d435_link"/>
+  <link name="rs_d435_link">
+    <inertial>
+      <origin xyz="0 0 0"/>
+      <mass value="0.1"/>
+      <inertia ixx="0.01" ixy="0" ixz="0"
+               iyy="0.01" iyz="0"
+               izz="0.01" />
+    </inertial>
+  </link>
+  <transmission name="tran1">
+    <type>transmission_interface/SimpleTransmission</type>
+    <joint name="joint1">
+      <hardwareInterface>hardware_interface/EffortJointInterface</hardwareInterface>
+    </joint>
+    <actuator name="motor1">
+      <hardwareInterface>hardware_interface/EffortJointInterface</hardwareInterface>
+      <mechanicalReduction>1</mechanicalReduction>
+    </actuator>
+  </transmission>
     <!-- camera depth joints and links -->
   <joint name="rs_d435_depth_joint" type="fixed">
